Commit message: Now testing collision detection. Self collisions seem to work

File: grippers/franka_gripper.urdf (robot description, URDF)
Before this commit: robot panda, 15 links, 14 joints
Links:
- link panda_leftfinger: geometry collision mesh filename=meshes/finger.stl; visual mesh filename=meshes/finger.stl
- link panda_rightfinger: geometry collision mesh filename=meshes/finger.stl; visual mesh filename=meshes/finger.stl
